Commit message: Added ABU 2027 map, updated robot dimention and updated cartographer launch file.
Signed-off-by: Tin LetHax <thipok17@gmail.com>

File: R1/description_r1/robot_core_r1.xacro (robot description, xacro)
@@ -33,5 +33,5 @@
 			<origin xyz="0 0 0.1"/>
 			<geometry>
-				<cylinder radius="0.4" length="1.2"/>
+				<box size="0.7 0.7 0.7"/>
 			</geometry>
 			<material name="green"/>
@@ -40,5 +40,5 @@
 			<origin xyz="0 0 0.2"/>
 			<geometry>
-				<cylinder radius="0.4" length="1.2"/>
+				<box size="0.7 0.7 0.7"/>
 			</geometry>
 		</collision>
@@ -174,5 +174,5 @@
     <parent link="base_link_r1"/>
     <child link="lidar_link_1_r1"/>
-    <origin xyz="0.35 0 0.03" rpy="0 0 0"/>
+    <origin xyz="0.30 0.30 0.03" rpy="0 0 0"/>
   </joint>
   <gazebo reference="lidar_link_1_r1">
@@ -184,7 +184,7 @@
         <scan>
           <horizontal>
-            <samples>720</samples>
-            <min_angle>-1.57</min_angle>
-            <max_angle>1.57</max_angle>
+            <samples>800</samples>
+            <min_angle>-1.745329</min_angle>
+            <max_angle>1.745329</max_angle>
           </horizontal>
         </scan>
@@ -225,5 +225,5 @@
     <parent link="base_link_r1"/>
     <child link="lidar_link_2_r1"/>
-	<origin xyz="-0.35 0 0.03" rpy="0 0 3.141593"/>
+	<origin xyz="-0.30 -0.30 0.03" rpy="0 0 3.141593"/>
   </joint>
   <gazebo reference="lidar_link_2_r1">
@@ -235,7 +235,7 @@
         <scan>
           <horizontal>
-            <samples>250</samples>
-            <min_angle>-1.57</min_angle>
-            <max_angle>1.57</max_angle>
+            <samples>800</samples>
+            <min_angle>-1.745329</min_angle>
+            <max_angle>1.745329</max_angle>
           </horizontal>
         </scan>
